Commit message: joints

File: demos/urdf/rrbot.urdf (robot description, URDF)
Before this commit: robot rrbot, 3 links, 2 joints
Links:
- removed link base_link
- link link1: mass 1.0 -> 1; geometry collision box size=0.1 0.1 2; visual box size=0.1 0.1 2
- link link2: mass 1.0 -> 1; geometry collision box size=0.1 0.1 1; visual box size=0.1 0.1 1
Joints:
- removed joint joint_1
- removed joint joint_2
- added joint joint1: type revolute, parent link1, child link2, origin xyz=0 0.1 1.95 rpy=0 0 0, axis 0 1 0, limit lower=-10000000000000000 upper=10000000000000000 effort=1000 velocity=10
